File: Sch/Power_relay_control.kicad_sch (KiCad schematic)
At the start: 16 parts, among them U7 PC817, U8 PC817

Commit message: VER1.0: плата разведена, файлы по плате готовы
Parts:
- C74: Description P/N (none) -> Capacitor SMD 50V
- J8: Purpose Precharge -> (none)
- J9: Purpose Relay_1 -> (none)
- R60, R61, R62, R63, R64, R65: Description P/N (none) -> Resistor SMD
- U7, U8: value PC817 -> (none); Description P/N (none) -> Optocoupler; Product Name (none) -> PC817
Changed lines of the file:
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@@
-			)
-		)
-		(property "Purpose" ""
-			(at 161.925 78.74 0)
-			(hide yes)
-			(show_name no)
-			(do_not_autoplace no)
-			(effects
-				(font
-					(size 1.27 1.27)
-				)
 			)
 		)
@@
 			)
 		)
-		(property "Value" "PC817"
+		(property "Value" ""
 			(at 140.97 93.98 0)
 			(show_name no)
@@
 		)
 		(property "Description" "DC Optocoupler, Vce 35V, CTR 50-300%, DIP-4"
+			(at 140.97 88.9 0)
+			(hide yes)
+			(show_name no)
+			(do_not_autoplace no)
+			(effects
+				(font
+					(size 1.27 1.27)
+				)
+			)
+		)
+		(property "Description P/N" "Optocoupler"
+			(at 140.97 88.9 0)
+			(hide yes)
+			(show_name no)
+			(do_not_autoplace no)
+			(effects
+				(font
+					(size 1.27 1.27)
+				)
+			)
+		)
+		(property "Product Name" "PC817"
 			(at 140.97 88.9 0)
 			(hide yes)
@@
 			)
 		)
-		(property "Purpose" ""
-			(at 130.81 127 0)
-			(hide yes)
-			(show_name no)
-			(do_not_autoplace no)
-			(effects
-				(font
-					(size 1.27 1.27)
-				)
-			)
-		)
-		(property "Description P/N" ""
+		(property "Description P/N" "Resistor SMD"
 			(at 130.81 127 0)
 			(hide yes)
@@
 			)
 		)
-		(property "Purpose" ""
-			(at 186.055 92.71 0)
-			(hide yes)
-			(show_name no)
-			(do_not_autoplace no)
-			(effects
-				(font
-					(size 1.27 1.27)
-				)
-			)
-		)
 		(property "Description P/N" "Blue LED"
 			(at 186.055 92.71 0)
@@
 			)
 		)
-		(property "Purpose" ""
-			(at 162.56 91.44 0)
-			(hide yes)
-			(show_name no)
-			(do_not_autoplace no)
-			(effects
-				(font
-					(size 1.27 1.27)
-				)
-			)
-		)
 		(property "Description P/N" "Self-Protected Low Side Driver with Temperature and Current Limit, SOT−223"
 			(at 162.56 91.44 0)
@@
 		(property "Replacement" ""
 			(at 121.92 127 0)
-			(hide yes)
-			(show_name no)
-			(do_not_autoplace no)
-			(effects
-				(font
-					(size 1.27 1.27)
-				)
-			)
-		)
-		(property "Purpose" "Relay_1"
-			(at 121.92 121.92 0)
 			(hide yes)
 			(show_name no)
@@
 			)
 		)
-		(property "Value" "PC817"
+		(property "Value" ""
 			(at 140.97 134.62 0)
 			(show_name no)
@@
 		)
 		(property "Description" "DC Optocoupler, Vce 35V, CTR 50-300%, DIP-4"
+			(at 140.97 129.54 0)
+			(hide yes)
+			(show_name no)
+			(do_not_autoplace no)
+			(effects
+				(font
+					(size 1.27 1.27)
+				)
+			)
+		)
+		(property "Description P/N" "Optocoupler"
+			(at 140.97 129.54 0)
+			(hide yes)
+			(show_name no)
+			(do_not_autoplace no)
+			(effects
+				(font
+					(size 1.27 1.27)
+				)
+			)
+		)
+		(property "Product Name" "PC817"
 			(at 140.97 129.54 0)
 			(hide yes)
@@
 			)
 		)
-		(property "Purpose" ""
-			(at 151.13 134.62 0)
-			(hide yes)
-			(show_name no)
-			(do_not_autoplace no)
-			(effects
-				(font
-					(size 1.27 1.27)
-				)
-			)
-		)
-		(property "Description P/N" ""
+		(property "Description P/N" "Resistor SMD"
 			(at 151.13 134.62 0)
 			(hide yes)
@@
 			)
 		)
-		(property "Purpose" "Precharge"
-			(at 191.135 72.898 0)
-			(hide yes)
-			(show_name no)
-			(do_not_autoplace no)
-			(effects
-				(font
-					(size 1.27 1.27)
-				)
-			)
-		)
 		(property "Description P/N" "Connector"
 			(at 191.135 78.74 0)
@@
 			)
 		)
-		(property "Purpose" ""
-			(at 157.48 127 0)
-			(hide yes)
-			(show_name no)
-			(do_not_autoplace no)
-			(effects
-				(font
-					(size 1.27 1.27)
-				)
-			)
-		)
 		(property "Description P/N" "Schottky barrier diode"
 			(at 157.48 127 0)
@@
 			)
 		)
-		(property "Purpose" ""
-			(at 127 134.62 0)
-			(hide yes)
-			(show_name no)
-			(do_not_autoplace no)
-			(effects
-				(font
-					(size 1.27 1.27)
-				)
-			)
-		)
-		(property "Description P/N" ""
+		(property "Description P/N" "Resistor SMD"
 			(at 127 134.62 0)
 			(hide yes)
@@
 			)
 		)
-		(property "Purpose" ""
-			(at 149.86 96.52 0)
-			(hide yes)
-			(show_name no)
-			(do_not_autoplace no)
-			(effects
-				(font
-					(size 1.27 1.27)
-				)
-			)
-		)
-		(property "Description P/N" ""
+		(property "Description P/N" "Resistor SMD"
 			(at 149.86 96.52 0)
 			(hide yes)
@@
 			)
 		)
-		(property "Purpose" ""
-			(at 157.48 134.62 0)
-			(hide yes)
-			(show_name no)
-			(do_not_autoplace no)
-			(effects
-				(font
-					(size 1.27 1.27)
-				)
-			)
-		)
-		(property "Description P/N" ""
+		(property "Description P/N" "Capacitor SMD 50V"
 			(at 157.48 134.62 0)
 			(hide yes)
@@
 		)
 		(property "Replacement" ""
-			(at 127 129.54 0)
-			(hide yes)
-			(show_name no)
-			(do_not_autoplace no)
-			(effects
-				(font
-					(size 1.27 1.27)
-				)
-			)
-		)
-		(property "Purpose" ""
 			(at 127 129.54 0)
 			(hide yes)
@@
 			)
 		)
-		(property "Purpose" ""
-			(at 130.81 86.36 0)
-			(hide yes)
-			(show_name no)
-			(do_not_autoplace no)
-			(effects
-				(font
-					(size 1.27 1.27)
-				)
-			)
-		)
-		(property "Description P/N" ""
+		(property "Description P/N" "Resistor SMD"
 			(at 130.81 86.36 0)
 			(hide yes)
@@
 			)
 		)
-		(property "Purpose" ""
+		(property "Description P/N" "Resistor SMD"
 			(at 186.055 87.63 0)
 			(hide yes)
-			(show_name no)
-			(do_not_autoplace no)
-			(effects
-				(font
-					(size 1.27 1.27)
-				)
-			)
-		)
-		(property "Description P/N" ""
-			(at 186.055 87.63 0)
-			(hide yes)
