File: Sch/Voltage_measure.kicad_sch (KiCad schematic)
At the start: 31 parts, among them U6 OPA333xxDBV

Commit message: VER1.0: оптимизировал схему измерения напряжения
Parts:
- R25, R26, R27: footprint Resistor_SMD:R_1206_3216Metric -> Resistor_SMD:R_2512_6332Metric_Pad1.40x3.35mm_HandSolder
- R5, R9: value 16k -> 8k
Changed lines of the file:
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@@
 			)
 		)
-		(property "Footprint" "Resistor_SMD:R_1206_3216Metric"
+		(property "Footprint" "Resistor_SMD:R_2512_6332Metric_Pad1.40x3.35mm_HandSolder"
 			(at 69.342 78.74 90)
 			(hide yes)
@@
 			)
 		)
+		(property "Function" ""
+			(at 71.12 78.74 0)
+			(hide yes)
+			(show_name no)
+			(do_not_autoplace no)
+			(effects
+				(font
+					(size 1.27 1.27)
+				)
+			)
+		)
 		(pin "1"
 		)
@@
 			)
 		)
-		(property "Footprint" "Resistor_SMD:R_1206_3216Metric"
+		(property "Footprint" "Resistor_SMD:R_2512_6332Metric_Pad1.40x3.35mm_HandSolder"
 			(at 69.342 71.12 90)
 			(hide yes)
@@
 			)
 		)
+		(property "Function" ""
+			(at 71.12 71.12 0)
+			(hide yes)
+			(show_name no)
+			(do_not_autoplace no)
+			(effects
+				(font
+					(size 1.27 1.27)
+				)
+			)
+		)
 		(pin "1"
 		)
@@
 			)
 		)
-		(property "Value" "16k"
+		(property "Value" "8k"
 			(at 109.22 96.52 90)
 			(show_name no)
@@
 			)
 		)
-		(property "Footprint" "Resistor_SMD:R_1206_3216Metric"
+		(property "Footprint" "Resistor_SMD:R_2512_6332Metric_Pad1.40x3.35mm_HandSolder"
 			(at 69.342 86.36 90)
 			(hide yes)
@@
 			)
 		)
+		(property "Function" ""
+			(at 71.12 86.36 0)
+			(hide yes)
+			(show_name no)
+			(do_not_autoplace no)
+			(effects
+				(font
+					(size 1.27 1.27)
+				)
+			)
+		)
 		(pin "1"
 		)
@@
 		(dnp no)
 		(property "Reference" "R5"
-			(at 99.568 89.916 90)
+			(at 99.568 88.9 90)
 			(show_name no)
 			(do_not_autoplace no)
@@
 					(size 1.27 1.27)
 				)
-				(justify right)
 			)
 		)
-		(property "Value" "16k"
-			(at 101.6 89.662 90)
+		(property "Value" "8k"
+			(at 101.6 88.9 90)
 			(show_name no)
 			(do_not_autoplace no)
@@
 					(size 1.27 1.27)
 				)
-				(justify right)
 			)
 		)
@@
 		(property "Value" "OPA333xxDBV"
 			(at 193.04 101.346 0)
+			(hide yes)
 			(show_name no)
 			(do_not_autoplace no)
@@
 			)
 		)
+		(property "Product Name" ""
+			(at 190.5 96.52 0)
+			(hide yes)
+			(show_name no)
+			(do_not_autoplace no)
+			(effects
+				(font
+					(size 1.27 1.27)
+				)
+			)
+		)
+		(property "Description P/N" ""
+			(at 190.5 96.52 0)
+			(hide yes)
+			(show_name no)
+			(do_not_autoplace no)
+			(effects
+				(font
+					(size 1.27 1.27)
+				)
+			)
+		)
+		(property "Replacement" ""
+			(at 190.5 96.52 0)
+			(hide yes)
+			(show_name no)
+			(do_not_autoplace no)
+			(effects
+				(font
+					(size 1.27 1.27)
+				)
+			)
+		)
+		(property "Function" ""
+			(at 190.5 96.52 0)
+			(hide yes)
+			(show_name no)
+			(do_not_autoplace no)
+			(effects
+				(font
+					(size 1.27 1.27)
+				)
+			)
+		)
 		(pin "2"
 		)
@@
 	)
 	(symbol
-		(lib_id "power:+3.3V")
-		(at 146.05 92.71 0)
+		(lib_id "power:+1V0")
+		(at 101.6 85.09 0)
 		(unit 1)
 		(body_style 1)
@@
 		(in_pos_files yes)
 		(dnp no)
-		(fields_autoplaced yes)
-		(property "Reference" "#PWR017"
-			(at 146.05 96.52 0)
+		(property "Reference" "#PWR0232"
+			(at 101.6 88.9 0)
 			(hide yes)
 			(show_name no)
@@
 			)
 		)
-		(property "Value" "+3.3V"
-			(at 146.05 88.9 0)
+		(property "Value" "+1V0"
+			(at 101.6 81.28 0)
 			(show_name no)
 			(do_not_autoplace no)
@@
 		)
 		(property "Footprint" ""
-			(at 146.05 92.71 0)
+			(at 101.6 85.09 0)
 			(hide yes)
 			(show_name no)
@@
 		)
 		(property "Datasheet" ""
-			(at 146.05 92.71 0)
+			(at 101.6 85.09 0)
 			(hide yes)
 			(show_name no)
@@
 			)
 		)
-		(property "Description" ""
-			(at 146.05 92.71 0)
+		(property "Description" "Power symbol creates a global label with name \"+1V0\""
+			(at 101.6 85.09 0)
 			(hide yes)
 			(show_name no)
@@
 			(project "PDU_Container_MCU_PCB"
 				(path "/7b040528-7065-4d6b-8722-075d9f593d01/3921ac16-82e1-4ab7-a80c-f6d04f7998f3"
-					(reference "#PWR017")
+					(reference "#PWR0232")
 					(unit 1)
 				)
 				(path "/7b040528-7065-4d6b-8722-075d9f593d01/93ce951f-aa44-4957-b9af-2a48ec1cc942"
-					(reference "#PWR0110")
+					(reference "#PWR0234")
 					(unit 1)
 				)
 				(path "/7b040528-7065-4d6b-8722-075d9f593d01/a8507d04-f082-4072-a7b5-a924f1d0a9fd"
-					(reference "#PWR078")
+					(reference "#PWR0233")
 					(unit 1)
 				)
@@
 	)
 	(symbol
-		(lib_id "power:+1V0")
-		(at 101.6 85.09 0)
+		(lib_id "power:+3.3V")
+		(at 146.05 92.71 0)
 		(unit 1)
 		(body_style 1)
@@
 		(in_pos_files yes)
 		(dnp no)
-		(property "Reference" "#PWR09"
-			(at 101.6 88.9 0)
+		(fields_autoplaced yes)
+		(property "Reference" "#PWR017"
+			(at 146.05 96.52 0)
 			(hide yes)
 			(show_name no)
@@
 			)
 		)
-		(property "Value" "+1V0"
-			(at 101.346 81.534 0)
+		(property "Value" "+3.3V"
+			(at 146.05 88.9 0)
 			(show_name no)
 			(do_not_autoplace no)
@@
 		)
 		(property "Footprint" ""
-			(at 101.6 85.09 0)
+			(at 146.05 92.71 0)
 			(hide yes)
 			(show_name no)
@@
 		)
 		(property "Datasheet" ""
-			(at 101.6 85.09 0)
+			(at 146.05 92.71 0)
 			(hide yes)
 			(show_name no)
@@
 			)
 		)
-		(property "Description" "Power symbol creates a global label with name \"+1V0\""
-			(at 101.6 85.09 0)
+		(property "Description" ""
+			(at 146.05 92.71 0)
 			(hide yes)
 			(show_name no)
@@
 			(project "PDU_Container_MCU_PCB"
 				(path "/7b040528-7065-4d6b-8722-075d9f593d01/3921ac16-82e1-4ab7-a80c-f6d04f7998f3"
-					(reference "#PWR09")
+					(reference "#PWR017")
 					(unit 1)
 				)
 				(path "/7b040528-7065-4d6b-8722-075d9f593d01/93ce951f-aa44-4957-b9af-2a48ec1cc942"
-					(reference "#PWR0108")
+					(reference "#PWR0110")
 					(unit 1)
 				)
 				(path "/7b040528-7065-4d6b-8722-075d9f593d01/a8507d04-f082-4072-a7b5-a924f1d0a9fd"
-					(reference "#PWR076")
+					(reference "#PWR078")
 					(unit 1)
 				)

Commit message: VER1.0: плата разведена, файлы по плате готовы
Parts:
- C1, C10, C12, C2, C22, C23, C24, C25, C9: Description P/N (none) -> Capacitor SMD 50V
- D6: value TO-3216BC-MYF -> (none); Description P/N (none) -> Yellow LED; Product Name (none) -> TO-3216BC-MYF
- D7: value S1M -> (none); Description P/N (none) -> Diode; Product Name (none) -> S1M
- J3: Purpose VDC+ -> (none)
- J7: Purpose GNDPWR -> (none)
- R1, R10, R13, R2, R21, R25, R26, R27, R3, R4, R5, R6, R7, R8, R9: Description P/N (none) -> Resistor SMD
- U6: value OPA333xxDBV -> (none); Description P/N (none) -> Op-Amp; Product Name (none) -> OPA333xxDBV
