File: Sch/Voltage_measure.kicad_sch (KiCad schematic)
At the start: 31 parts

Commit message: VER1.0: обновил гербера и BOM
Parts:
- C10: value 0.27u -> 220n
- C23, C25: value 0.1u -> 100n
- R1, R13, R2, R21, R25, R26, R27, R3, R4, R5, R6, R7, R8, R9: Description P/N Resistor SMD -> Resistor SMD 1%
- R10: value 49.9 -> 120; Description P/N Resistor SMD -> Resistor SMD 1%
- U6: Product Name OPA333xxDBV -> OPA333
Changed lines of the file:
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@@
 			)
 		)
-		(property "Description P/N" "Resistor SMD"
+		(property "Description P/N" "Resistor SMD 1%"
 			(at 71.12 78.74 0)
 			(hide yes)
@@
 			)
 		)
-		(property "Description P/N" "Resistor SMD"
+		(property "Description P/N" "Resistor SMD 1%"
 			(at 161.29 99.06 0)
 			(hide yes)
@@
 			)
 		)
-		(property "Value" "0.27u"
+		(property "Value" "220n"
 			(at 216.281 104.5722 0)
 			(show_name no)
@@
 			)
 		)
-		(property "Description P/N" "Resistor SMD"
+		(property "Description P/N" "Resistor SMD 1%"
 			(at 167.64 106.68 0)
 			(hide yes)
@@
 			)
 		)
-		(property "Value" "0.1u"
+		(property "Value" "100n"
 			(at 153.035 117.475 0)
 			(show_name no)
@@
 		(fields_autoplaced yes)
 		(property "Reference" "R10"
-			(at 207.01 91.8042 90)
+			(at 207.01 90.17 90)
 			(show_name no)
 			(do_not_autoplace no)
@@
 			)
 		)
-		(property "Value" "49.9"
-			(at 207.01 94.3411 90)
+		(property "Value" "120"
+			(at 207.01 92.71 90)
 			(show_name no)
 			(do_not_autoplace no)
@@
 			)
 		)
-		(property "Description P/N" "Resistor SMD"
+		(property "Description P/N" "Resistor SMD 1%"
 			(at 207.01 96.52 0)
 			(hide yes)
@@
 			)
 		)
-		(property "Description P/N" "Resistor SMD"
+		(property "Description P/N" "Resistor SMD 1%"
 			(at 97.79 76.2 0)
 			(hide yes)
@@
 			)
 		)
-		(property "Description P/N" "Resistor SMD"
+		(property "Description P/N" "Resistor SMD 1%"
 			(at 71.12 71.12 0)
 			(hide yes)
@@
 			)
 		)
-		(property "Description P/N" "Resistor SMD"
+		(property "Description P/N" "Resistor SMD 1%"
 			(at 109.22 96.52 0)
 			(hide yes)
@@
 			)
 		)
-		(property "Description P/N" "Resistor SMD"
+		(property "Description P/N" "Resistor SMD 1%"
 			(at 109.22 88.9 0)
 			(hide yes)
@@
 			)
 		)
-		(property "Description P/N" "Resistor SMD"
+		(property "Description P/N" "Resistor SMD 1%"
 			(at 161.29 93.98 0)
 			(hide yes)
@@
 			)
 		)
-		(property "Description P/N" "Resistor SMD"
+		(property "Description P/N" "Resistor SMD 1%"
 			(at 167.64 85.725 0)
 			(hide yes)
@@
 			)
 		)
-		(property "Description P/N" "Resistor SMD"
+		(property "Description P/N" "Resistor SMD 1%"
 			(at 71.12 86.36 0)
 			(hide yes)
@@
 			)
 		)
-		(property "Description P/N" "Resistor SMD"
+		(property "Description P/N" "Resistor SMD 1%"
 			(at 101.6 88.9 0)
 			(hide yes)
@@
 			)
 		)
-		(property "Value" "0.1u"
+		(property "Value" "100n"
 			(at 128.905 117.475 0)
 			(show_name no)
@@
 			)
 		)
-		(property "Description P/N" "Resistor SMD"
+		(property "Description P/N" "Resistor SMD 1%"
 			(at 105.41 76.2 0)
 			(hide yes)
@@
 			)
 		)
-		(property "Product Name" "OPA333xxDBV"
+		(property "Product Name" "OPA333"
 			(at 190.5 96.52 0)
 			(hide yes)
@@
 			)
 		)
-		(property "Description P/N" "Resistor SMD"
+		(property "Description P/N" "Resistor SMD 1%"
 			(at 115.57 92.71 0)
 			(hide yes)
@@
 			)
 		)
-		(property "Description P/N" "Resistor SMD"
+		(property "Description P/N" "Resistor SMD 1%"
 			(at 109.22 81.28 0)
 			(hide yes)
