File: Sch/Current_measure.kicad_sch (KiCad schematic)
At the start: 22 parts, among them Q7 BC847, Q9 BC857, U2 OPA333xxDBV

Commit message: VER1.0: добавил функционалку и расставил все на плате
Parts:
- R56: footprint Resistor_SMD:R_0805_2012Metric_Pad1.20x1.40mm_HandSolder -> Resistor_SMD:R_2512_6332Metric_Pad1.40x3.35mm_HandSolder
Changed lines of the file:
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@@
 			)
 		)
-		(property "Footprint" "Resistor_SMD:R_0805_2012Metric_Pad1.20x1.40mm_HandSolder"
+		(property "Footprint" "Resistor_SMD:R_2512_6332Metric_Pad1.40x3.35mm_HandSolder"
 			(at 110.998 101.6 90)
 			(hide yes)
@@
 			(at 109.22 101.6 0)
 			(hide yes)
+			(show_name no)
+			(do_not_autoplace no)
+			(effects
+				(font
+					(size 1.27 1.27)
+				)
+			)
+		)
+		(property "Function" ""
+			(at 109.22 101.6 0)
+			(hide yes)

Commit message: VER1.0: плата разведена
Connections:
- net +15V: now also J16.1 (Pin_1); no longer J16.3 (Pin_3)
- net -15V: now also J16.2 (Pin_2); no longer J16.1 (Pin_1)
- net M: now also J16.3 (Pin_3); no longer J16.4 (Pin_4)
- net Current_SENSE renamed Current_measure
Other:
- moved on the sheet: J16
Changed lines of the file:
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@@
 	)
 	(no_connect
-		(at 96.52 95.25)
+		(at 88.9 100.33)
 	)
 	(wire
@@
 	(wire
 		(pts
-			(xy 190.5 72.39) (xy 190.5 74.93)
+			(xy 101.6 95.25) (xy 109.22 95.25)
 		)
 		(stroke
@@
 	(wire
 		(pts
-			(xy 96.52 107.95) (xy 93.98 107.95)
+			(xy 190.5 72.39) (xy 190.5 74.93)
 		)
 		(stroke
@@
 	(wire
 		(pts
-			(xy 99.06 107.95) (xy 101.6 107.95)
-		)
-		(stroke
-			(width 0)
-			(type default)
-		)
-	)
-	(wire
-		(pts
 			(xy 130.81 156.21) (xy 130.81 157.48)
 		)
@@
 	(wire
 		(pts
-			(xy 99.06 95.25) (xy 109.22 95.25)
+			(xy 176.53 160.02) (xy 186.69 160.02)
 		)
 		(stroke
@@
 	(wire
 		(pts
-			(xy 176.53 160.02) (xy 186.69 160.02)
+			(xy 101.6 149.86) (xy 105.41 149.86)
 		)
 		(stroke
@@
 	(wire
 		(pts
-			(xy 101.6 149.86) (xy 105.41 149.86)
+			(xy 99.06 148.59) (xy 99.06 149.86)
 		)
 		(stroke
@@
 	(wire
 		(pts
-			(xy 99.06 148.59) (xy 99.06 149.86)
+			(xy 176.53 147.32) (xy 186.69 147.32)
 		)
 		(stroke
@@
 	(wire
 		(pts
-			(xy 176.53 147.32) (xy 186.69 147.32)
+			(xy 101.6 95.25) (xy 101.6 100.33)
 		)
 		(stroke
@@
 	)
 	(label "+15V"
-		(at 101.6 107.95 0)
+		(at 101.6 102.87 0)
 		(effects
 			(font
@@
 	)
 	(label "-15V"
-		(at 93.98 107.95 180)
+		(at 88.9 102.87 180)
 		(effects
 			(font
@@
 		)
 	)
-	(global_label "Current_SENSE"
+	(hierarchical_label "Current_measure"
 		(shape output)
 		(at 194.31 62.23 0)
-		(fields_autoplaced yes)
 		(effects
 			(font
@@
 			(justify left)
 		)
-		(property "Intersheetrefs" "${INTERSHEET_REFS}"
-			(at 211.265 62.23 0)
-			(hide yes)
-			(show_name no)
-			(do_not_autoplace no)
-			(effects
-				(font
-					(size 1.27 1.27)
-				)
-				(justify left)
-			)
-		)
 	)
 	(symbol
@@
 	(symbol
 		(lib_id "Connector_Generic:Conn_02x02_Odd_Even")
-		(at 96.52 102.87 90)
+		(at 96.52 102.87 180)
 		(unit 1)
 		(body_style 1)
@@
 		(dnp no)
 		(property "Reference" "J16"
-			(at 102.362 101.346 90)
+			(at 94.996 97.79 0)
 			(show_name no)
 			(do_not_autoplace no)
@@
 		)
 		(property "Value" ""
-			(at 92.71 101.6 0)
+			(at 95.25 106.68 0)
 			(hide yes)
 			(show_name no)
@@
 		)
 		(property "Function" "Current Sensor"
-			(at 87.63 101.6 90)
+			(at 95.758 105.918 0)
 			(show_name no)
 			(do_not_autoplace no)

Commit message: VER1.0: плата разведена, файлы по плате готовы
Parts:
- C14, C20, C7, C70: Description P/N (none) -> Capacitor SMD 50V
- D21: Description P/N (none) -> DC/DC; Product Name (none) -> UWE1215S-3WR3
- L5: Description P/N (none) -> Inductor common mode SMD
- Q7: value BC847 -> (none); Description P/N (none) -> Bipolar N; Product Name (none) -> BC847
- Q9: value BC857 -> (none); Description P/N (none) -> Bipolar P; Product Name (none) -> BC857
- R18, R56, R88, R90: Description P/N (none) -> Resistor SMD
- U2: value OPA333xxDBV -> (none); Description P/N (none) -> Op-Amp; Product Name (none) -> OPA333xxDBV
Changed lines of the file:
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@@
 			)
 		)
-		(property "Purpose" ""
-			(at 190.5 68.58 0)
-			(hide yes)
-			(show_name no)
-			(do_not_autoplace no)
-			(effects
-				(font
-					(size 1.27 1.27)
-				)
-			)
-		)
-		(property "Description P/N" ""
+		(property "Description P/N" "Capacitor SMD 50V"
 			(at 190.5 68.58 0)
 			(hide yes)
@@
 			)
 		)
-		(property "Purpose" ""
-			(at 137.16 116.84 0)
-			(hide yes)
-			(show_name no)
-			(do_not_autoplace no)
-			(effects
-				(font
-					(size 1.27 1.27)
-				)
-			)
-		)
-		(property "Description P/N" ""
+		(property "Description P/N" "Capacitor SMD 50V"
 			(at 137.16 116.84 0)
 			(hide yes)
@@
 			)
 		)
-		(property "Value" "BC857"
+		(property "Value" ""
 			(at 193.04 113.0299 0)
 			(show_name no)
@@
 			)
 		)
+		(property "Description P/N" "Bipolar P"
+			(at 187.96 111.76 0)
+			(hide yes)
+			(show_name no)
+			(do_not_autoplace no)
+			(effects
+				(font
+					(size 1.27 1.27)
+				)
+			)
+		)
+		(property "Product Name" "BC857"
+			(at 187.96 111.76 0)
+			(hide yes)
+			(show_name no)
+			(do_not_autoplace no)
+			(effects
+				(font
+					(size 1.27 1.27)
+				)
+			)
+		)
 		(pin "1"
 		)
@@
 			)
 		)
-		(property "Purpose" ""
-			(at 190.5 57.15 0)
-			(hide yes)
-			(show_name no)
-			(do_not_autoplace no)
-			(effects
-				(font
-					(size 1.27 1.27)
-				)
-			)
-		)
 		(property "Description P/N" "Schottky barrier diode"
 			(at 190.5 57.15 0)
@@
 			)
 		)
-		(property "Purpose" ""
-			(at 125.73 92.71 0)
-			(hide yes)
-			(show_name no)
-			(do_not_autoplace no)
-			(effects
-				(font
-					(size 1.27 1.27)
-				)
-			)
-		)
-		(property "Description P/N" ""
+		(property "Description P/N" "Capacitor SMD 50V"
 			(at 125.73 92.71 0)
 			(hide yes)
@@
 			)
 		)
-		(property "Description P/N" ""
+		(property "Description P/N" "Inductor common mode SMD"
 			(at 125.73 153.67 0)
 			(hide yes)
@@
 			)
 		)
-		(property "Purpose" ""
-			(at 162.56 93.98 0)
-			(hide yes)
-			(show_name no)
-			(do_not_autoplace no)
-			(effects
-				(font
-					(size 1.27 1.27)
-				)
-			)
-		)
-		(property "Description P/N" ""
+		(property "Description P/N" "Capacitor SMD 50V"
 			(at 162.56 93.98 0)
 			(hide yes)
@@
 			)
 		)
-		(property "Purpose" ""
-			(at 133.35 92.71 0)
-			(hide yes)
-			(show_name no)
-			(do_not_autoplace no)
-			(effects
-				(font
-					(size 1.27 1.27)
-				)
-			)
-		)
-		(property "Description P/N" ""
+		(property "Description P/N" "Resistor SMD"
 			(at 133.35 92.71 0)
 			(hide yes)
@@
 			)
 		)
-		(property "Datasheet" "UWE1215S-3WR3"
+		(property "Datasheet" ""
 			(at 158.75 146.05 0)
 			(hide yes)
@@
 			)
 		)
-		(property "Product Name" ""
+		(property "Product Name" "UWE1215S-3WR3"
 			(at 158.75 146.05 0)
 			(hide yes)
@@
 			)
 		)
-		(property "Description P/N" ""
+		(property "Description P/N" "DC/DC"
 			(at 158.75 146.05 0)
 			(hide yes)
@@
 			)
 		)
-		(property "Purpose" ""
-			(at 109.22 101.6 0)
-			(hide yes)
-			(show_name no)
-			(do_not_autoplace no)
-			(effects
-				(font
-					(size 1.27 1.27)
-				)
-			)
-		)
-		(property "Description P/N" ""
+		(property "Description P/N" "Resistor SMD"
 			(at 109.22 101.6 0)
 			(hide yes)
@@
 			)
 		)
-		(property "Purpose" ""
-			(at 184.15 62.23 0)
-			(hide yes)
-			(show_name no)
-			(do_not_autoplace no)
-			(effects
-				(font
-					(size 1.27 1.27)
-				)
-			)
-		)
-		(property "Description P/N" ""
+		(property "Description P/N" "Resistor SMD"
 			(at 184.15 62.23 0)
 			(hide yes)
@@
 			)
 		)
-		(property "Purpose" ""
-			(at 142.24 92.71 0)
-			(hide yes)
-			(show_name no)
-			(do_not_autoplace no)
-			(effects
-				(font
-					(size 1.27 1.27)
-				)
-			)
-		)
-		(property "Description P/N" ""
+		(property "Description P/N" "Resistor SMD"
 			(at 142.24 92.71 0)
 			(hide yes)
@@
 			)
 		)
-		(property "Value" "OPA333xxDBV"
+		(property "Value" ""
 			(at 160.02 108.966 0)
 			(hide yes)
@@
 			)
 		)
-		(property "Product Name" ""
+		(property "Product Name" "OPA333xxDBV"
 			(at 157.48 104.14 0)
 			(hide yes)
@@
 			)
 		)
-		(property "Description P/N" ""
+		(property "Description P/N" "Op-Amp"
 			(at 157.48 104.14 0)
 			(hide yes)
@@
 			)
 		)
-		(property "Value" "BC847"
+		(property "Value" ""
 			(at 193.04 97.7899 0)
 			(show_name no)
@@
 			(at 187.96 96.52 0)
 			(hide yes)
+			(show_name no)
+			(do_not_autoplace no)
+			(effects
+				(font
+					(size 1.27 1.27)
+				)
+			)
+		)
+		(property "Description P/N" "Bipolar N"
+			(at 187.96 96.52 0)
+			(hide yes)
+			(show_name no)
+			(do_not_autoplace no)
+			(effects
+				(font
+					(size 1.27 1.27)
+				)
+			)
+		)
+		(property "Product Name" "BC847"
+			(at 187.96 96.52 0)
+			(hide yes)

Commit message: VER1.0: поправил BOM
Parts:
- J16: Product Name DS1073-01-2x2MR3T6 -> DS1073-01-2x2-MVT6
Changed lines of the file:
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@@
 			)
 		)
-		(property "Product Name" "DS1073-01-2x2MR3T6"
+		(property "Product Name" "DS1073-01-2x2-MVT6"
 			(at 96.52 102.87 0)
 			(hide yes)
