File: Sch/Current_measure.kicad_sch (KiCad schematic)
At the start: 22 parts

Commit message: VER1.0: обновил гербера и BOM
Parts:
- R18, R88, R90: Description P/N Resistor SMD -> Resistor SMD 1%
- R56: Description P/N Resistor SMD -> Resistor SMD 0.1%
- U2: Product Name OPA333xxDBV -> OPA333
Changed lines of the file:
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@@
 			)
 		)
-		(property "Description P/N" "Resistor SMD"
+		(property "Description P/N" "Resistor SMD 1%"
 			(at 133.35 92.71 0)
 			(hide yes)
@@
 			)
 		)
-		(property "Description P/N" "Resistor SMD"
+		(property "Description P/N" "Resistor SMD 0.1%"
 			(at 109.22 101.6 0)
 			(hide yes)
@@
 			)
 		)
-		(property "Description P/N" "Resistor SMD"
+		(property "Description P/N" "Resistor SMD 1%"
 			(at 184.15 62.23 0)
 			(hide yes)
@@
 			)
 		)
-		(property "Description P/N" "Resistor SMD"
+		(property "Description P/N" "Resistor SMD 1%"
 			(at 142.24 92.71 0)
 			(hide yes)
@@
 			)
 		)
-		(property "Product Name" "OPA333xxDBV"
+		(property "Product Name" "OPA333"
 			(at 157.48 104.14 0)
 			(hide yes)
