File: PDU_Container_MCU_PCB.kicad_pcb (KiCad board)
At the start: 4 copper layers, 237.2 x 87.2 mm, 289 parts, among them Q10 BC857, Q7 BC847, Q8 BC847, Q9 BC857, U1 TLV431, U10 PC817, U11 PC817, U12 PC817, U13 PC817, U14 PC817, U15 HT75xx-1-SOT89, U2 OPA333xxDBV, U3 OPA333xxDBV, U31 TLV1117LV33DCYR, U32 OPA333xxDBV, U33 OPA333xxDBV, U4 TLV1117LV33DCYR, U6 OPA333xxDBV, U7 PC817, U8 PC817, U9 PC817

Commit message: VER1.0: добавил функционалку и расставил все на плате
Parts:
- removed C28, C29, C32, C33, C5: 100n, Capacitor_SMD:C_0805_2012Metric_Pad1.18x1.45mm_HandSolder
- removed C31: 4.7u, Capacitor_SMD:C_0805_2012Metric_Pad1.18x1.45mm_HandSolder
- removed C50, C51: 2.2u, Capacitor_SMD:C_0805_2012Metric_Pad1.18x1.45mm_HandSolder
- removed C6: 1u, Capacitor_SMD:C_0805_2012Metric_Pad1.18x1.45mm_HandSolder
- removed D13: ~, LED_SMD:LED_0805_2012Metric
- removed J2: ~, Connector_Molex:Molex_Mini-Fit_Jr_5566-04A_2x02_P4.20mm_Vertical
- removed R16, R17, R35, R36: 1k, Resistor_SMD:R_0805_2012Metric_Pad1.20x1.40mm_HandSolder
- removed TP1, TP2: TestPoint, TestPoint:TestPoint_Loop_D1.80mm_Drill1.0mm_Beaded
- added C13: 100n, Capacitor_SMD:C_0805_2012Metric_Pad1.18x1.45mm_HandSolder, B.Cu at (335.8, 206.2)
- added C15: 100n, Capacitor_SMD:C_0805_2012Metric_Pad1.18x1.45mm_HandSolder, B.Cu at (345.3, 208.2)
- added C21: 2.2u, Capacitor_SMD:C_0805_2012Metric_Pad1.18x1.45mm_HandSolder, B.Cu at (345.3, 203.8)
- added C65: 100n, Capacitor_SMD:C_0805_2012Metric_Pad1.18x1.45mm_HandSolder, B.Cu at (337.0, 212.0)
- added D42: ~, LED_SMD:LED_0805_2012Metric, F.Cu at (335.5, 217.2)
- added R11: 10k, Resistor_SMD:R_0805_2012Metric_Pad1.20x1.40mm_HandSolder, F.Cu at (331.5, 209.0)
- added R12: 1k, Resistor_SMD:R_0805_2012Metric_Pad1.20x1.40mm_HandSolder, B.Cu at (337.8, 217.2)
- added R14: 10k, Resistor_SMD:R_0805_2012Metric_Pad1.20x1.40mm_HandSolder, B.Cu at (339.3, 212.0)
- added R54: 20, Resistor_SMD:R_0805_2012Metric_Pad1.20x1.40mm_HandSolder, F.Cu at (325.5, 203.8)
- added R92: 1k, Resistor_SMD:R_0805_2012Metric_Pad1.20x1.40mm_HandSolder, B.Cu at (335.5, 217.2)
- added R95: 20, Resistor_SMD:R_0805_2012Metric_Pad1.20x1.40mm_HandSolder, F.Cu at (325.5, 206.2)
- added U16: ~, Package_TO_SOT_SMD:SOT-23-6, F.Cu at (329.6, 204.9)
- C11, C14, C20, C67, C7, C70, C80, C83, C87, C89, C90, C91, C92: moved to B.Cu
- C16: value 100n -> 4.7u
- C19: value 100n -> 1u
- C27: value 100n -> 2.2u
- C4: value 1u -> 100n
- R56, R87: footprint Resistor_SMD:R_0805_2012Metric_Pad1.20x1.40mm_HandSolder -> Resistor_SMD:R_2512_6332Metric_Pad1.40x3.35mm_HandSolder
- U5: footprint Package_QFP:LQFP-100_14x14mm_P0.5mm -> Package_QFP:LQFP-64_10x10mm_P0.5mm
- Y1: value ~ -> 16M
- moved C20 219.2 mm to (387.0, 244.2), turned to -90 degrees
- moved U2 210.3 mm to (383.2, 233.7), turned to 0 degrees
- moved D3 204.4 mm to (387.0, 240.2), turned to -90 degrees
- moved R18 199.6 mm to (387.0, 244.2), turned to 90 degrees
- moved C7 194.3 mm to (383.2, 233.7)
- moved C14 187.2 mm to (378.6, 233.2), turned to 0 degrees
- moved L6 177.0 mm to (244.8, 242.5), turned to -90 degrees
- moved D8 169.2 mm to (337.8, 217.2), turned to 90 degrees
- moved L7 168.3 mm to (255.0, 242.5), turned to 180 degrees
- moved C85 160.9 mm to (241.8, 242.5), turned to -90 degrees
- moved C86 155.8 mm to (247.8, 242.5), turned to 90 degrees
- moved C88 143.8 mm to (266.2, 244.9), turned to 90 degrees
- moved C87 141.8 mm to (263.2, 242.5), turned to 90 degrees
- moved D5 141.4 mm to (321.5, 197.0), turned to -90 degrees
- moved D23 127.5 mm to (283.2, 240.2)
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Connections:
- net +24V_SENSE renamed /GPIO3
- net Discete_1 renamed /RS_RXD_MCU
- net Discete_2 renamed /CAN_RXD_MCU
- net Discete_3 renamed /CAN_TXD_MCU
- net VDC_IN_SENSE renamed /GPIO2
- net VDC_OUT1_SENSE renamed /GPIO1
- C27 pad 1: +3.3V -> Net-(U5-VCAP_2)
- U5 pad 1: unconnected-(U5-PE2-Pad1) -> +3.3V
- U5 pad 10: GND -> unconnected-(U5-PC2-Pad10)
- U5 pad 11: +3.3V -> unconnected-(U5-PC3-Pad11)
- U5 pad 12: Net-(U5-PH0) -> GND
- U5 pad 13: Net-(U5-PH1) -> +3.3V
- U5 pad 14: NRST -> unconnected-(U5-PA0-Pad14)
- U5 pad 18: unconnected-(U5-PC3-Pad18) -> GND
- U5 pad 2: unconnected-(U5-PE3-Pad2) -> Net-(D42-A)
- U5 pad 20: GND -> unconnected-(U5-PA4-Pad20)
- U5 pad 21: +3.3V -> /ERROR_LvL1
- U5 pad 22: +3.3V -> /ERROR_LvL2
- U5 pad 23: unconnected-(U5-PA0-Pad23) -> /ERROR_LvL3
- U5 pad 27: GND -> unconnected-(U5-PB1-Pad27)
- U5 pad 28: +3.3V -> unconnected-(U5-PB2-Pad28)
- U5 pad 29: DAC_OUT1 -> unconnected-(U5-PB10-Pad29)
- U5 pad 3: unconnected-(U5-PE4-Pad3) -> Net-(D8-A)
- U5 pad 30: DAC_OUT2 -> unconnected-(U5-PB11-Pad30)
- U5 pad 31: Current_SENSE -> Net-(U5-VCAP_1)
- U5 pad 32: VDC_OUT2_SENSE -> +3.3V
- U5 pad 36: unconnected-(U5-PB1-Pad36) -> /GPIO4
- U5 pad 37: unconnected-(U5-PB2-Pad37) -> /GPIO5
- U5 pad 38: unconnected-(U5-PE7-Pad38) -> /GPIO6
- U5 pad 39: unconnected-(U5-PE8-Pad39) -> /GPIO7
- U5 pad 40: unconnected-(U5-PE9-Pad40) -> /GPIO8
- U5 pad 42: unconnected-(U5-PE11-Pad42) -> /RS_TXD_MCU
- U5 pad 46: Discete_4 -> /SWDIO
- U5 pad 47: unconnected-(U5-PB10-Pad47) -> Net-(U5-VCAP_2)
- U5 pad 48: unconnected-(U5-PB11-Pad48) -> +3.3V
- U5 pad 49: Net-(U5-VCAP_1) -> /SWCLK
- U5 pad 5: unconnected-(U5-PE6-Pad5) -> Net-(U5-PH0)
- U5 pad 50: +3.3V -> /Solenoid1_MCU
- U5 pad 51: unconnected-(U5-PB12-Pad51) -> /Solenoid2_MCU
- U5 pad 52: Net-(D8-A) -> /Solenoid3_MCU
- U5 pad 53: unconnected-(U5-PB14-Pad53) -> /Solenoid4_MCU
- U5 pad 57: Net-(D13-A) -> unconnected-(U5-PB5-Pad57)
- U5 pad 6: +3.3V -> Net-(U5-PH1)
- U5 pad 60: Shunt_2 -> BOOT0
- U5 pad 61: ~{Shunt_2_ON} -> unconnected-(U5-PB8-Pad61)
- U5 pad 62: Precharge_2 -> unconnected-(U5-PB9-Pad62)
- U5 pad 63: ~{Precharge_2_ON} -> GND
- U5 pad 64: Shunt_1 -> +3.3V
- U5 pad 7: unconnected-(U5-PC13-Pad7) -> NRST
Routing:
- net CAN1_TXD_MCU: track 22.7 -> 0.00 mm
- net CAN1_RXD_MCU: track 17.6 -> 0.00 mm
- net DAC_OUT1: track 10.3 -> 0.00 mm
- net DAC_OUT2: track 9.92 -> 0.00 mm
- net BOOT0: track 4.33 -> 0.00 mm
- net NRST: track 3.09 -> 0.00 mm
- net +3.3V: track 23.2 -> 22.7 mm
- removed copper zone on F.Cu, net GND

Commit message: VER1.0: оптимизировал схему измерения напряжения
Parts:
- removed R58: 1k, Resistor_SMD:R_0805_2012Metric_Pad1.20x1.40mm_HandSolder
- removed U1: TLV431, Package_TO_SOT_SMD:SOT-23
- added C5: 100n, Capacitor_SMD:C_0805_2012Metric_Pad1.18x1.45mm_HandSolder, B.Cu at (438.8, 171.5)
- added J35: ~, Connector_Molex:Molex_Mini-Fit_Jr_5566-04A_2x02_P4.20mm_Vertical, F.Cu at (262.8, 200.7)
- added U17: OPA333xxDBV, Package_TO_SOT_SMD:SOT-23-5, F.Cu at (438.8, 171.5)
- R132, R25, R26, R27, R28, R31, R34, R48, R51: footprint Resistor_SMD:R_1206_3216Metric -> Resistor_SMD:R_2512_6332Metric_Pad1.40x3.35mm_HandSolder
- R133, R137, R38, R44, R5, R9: value 16k -> 8k
- R23: value 240 -> 23.2k
- R24: value 1k -> 10k
- moved R133 14.4 mm to (427.5, 235.0), turned to 90 degrees
- moved R38 14.4 mm to (427.5, 215.0), turned to 90 degrees
- moved R5 14.4 mm to (427.5, 195.0), turned to 90 degrees
- moved D10 10.5 mm to (434.0, 213.5), turned to 180 degrees
- moved D6 10.5 mm to (434.0, 193.5), turned to 180 degrees
- moved D81 10.5 mm to (434.0, 233.5), turned to 180 degrees
- moved R135 6.72 mm to (430.2, 235.0), turned to -90 degrees
- moved R42 6.72 mm to (430.2, 215.0), turned to -90 degrees
- moved R7 6.72 mm to (430.2, 195.0), turned to -90 degrees
- moved C73 6.58 mm to (435.2, 171.5), turned to -90 degrees
- moved G*** 6.43 mm to (445.1, 173.5)
- moved R23 6.37 mm to (430.2, 171.5), turned to -90 degrees
- moved R27 5.98 mm to (445.0, 180.8)
- moved R28 5.98 mm to (445.0, 200.8)
- moved R48 5.98 mm to (445.0, 220.8)
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Connections:
- net CANH renamed /CANH
- net CANL renamed /CANL
- C73 pad 2: +1V0 -> Net-(U17-+)
- R23 pad 1: Net-(U1-K) -> +3.3VP
- R23 pad 2: +1V0 -> Net-(U17-+)
- R24 pad 1: +1V0 -> Net-(U17-+)
Routing:
- net +1V0: track 0.00 -> 81.3 mm, vias 0 -> 4
- net Net-(D40-A): track 0.00 -> 19.1 mm
- net Net-(D40-K): track 0.00 -> 17.9 mm
- net GNDPWR: track 67.5 -> 81.6 mm, vias 3 -> 19
- net GNDD: track 24.7 -> 38.6 mm, vias 0 -> 31
- net Net-(R38-Pad1): track 8.00 -> 16.5 mm
- net Net-(R5-Pad1): track 8.00 -> 16.5 mm
- net Net-(R133-Pad1): track 8.00 -> 16.5 mm
- net Net-(U17-+): track 0.00 -> 7.41 mm
- net +3.3VP: track 14.5 -> 20.5 mm, vias 3 -> 41
- net Net-(D19-Vin): track 0.00 -> 5.85 mm
- net Net-(D18-Vin): track 0.00 -> 5.77 mm
- net Net-(D18-CS): track 0.00 -> 5.05 mm
- net Net-(D82-VIN): track 12.3 -> 7.48 mm
- net Net-(D2-VIN): track 12.3 -> 7.48 mm
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- added copper zone on B.Cu, net +24V
- added copper zone on F.Cu, net +24V
- added copper zone on In2.Cu, net +24V
- added copper zone on F.Cu, net +3.3VP
- added copper zone on In2.Cu, net +3.3VP
- added copper zone on F.Cu, net -24V_IN
- added copper zone on B.Cu, net GNDD
- added copper zone on In1.Cu, net GNDD
- added copper zone on B.Cu, net GNDPWR
- added copper zone on F.Cu, net GNDPWR
- added copper zone on In1.Cu, net GNDPWR
- added copper zone on F.Cu, net Net-(D18-+Vo)
Other:
- outline, holes or cut-outs redrawn

Commit message: VER1.0: плата разведена
Parts:
- removed F2: ~, Fuse:Fuse_1812_4532Metric
- R88, R89, R90, R91: moved to B.Cu
- moved G*** 69.4 mm to (437.9, 242.5)
- moved G*** 67.5 mm to (437.9, 242.6)
- moved R89 54.8 mm to (358.5, 238.8), turned to 180 degrees
- moved R91 52.2 mm to (355.5, 239.8), turned to 90 degrees
- moved Q10 51.1 mm to (354.2, 239.8)
- moved Q8 51.1 mm to (358.0, 239.8), turned to -90 degrees
- moved C59 50.0 mm to (353.2, 239.8), turned to 90 degrees
- moved C11 42.2 mm to (350.0, 240.0)
- moved U3 42.2 mm to (350.0, 240.0), turned to 180 degrees
- moved C80 41.2 mm to (346.0, 240.0), turned to -90 degrees
- moved C81 41.1 mm to (277.4, 230.5)
- moved C82 41.1 mm to (283.4, 230.5)
- moved C83 41.1 mm to (298.9, 230.5)
- moved C84 41.1 mm to (301.9, 232.9)
- moved C89 41.1 mm to (322.6, 231.0)
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Connections:
- C10 pad 1: /Voltage_measure_1/VDC_SENSE -> /VDC_1_measure
- C20 pad 1: Current_SENSE -> /Current_1_measure
- C43 pad 1: /Voltage_measure_2/VDC_SENSE -> /VDC_2_measure
- C58 pad 1: /Voltage_measure_3/VDC_SENSE -> /VDC_3_measure
- C67 pad 1: Current_SENSE -> /Current_2_measure
- C68 pad 1: Net-(C68-Pad1) -> +24V
- C74 pad 1: /Relay_Control_1/Relay_FeedBack -> /Relay_FeedBack_1
- C75 pad 1: /Relay_Control_2/Relay_FeedBack -> /Relay_FeedBack_2
- C76 pad 1: /Relay_Control_3/Relay_FeedBack -> /Relay_FeedBack_3
- C77 pad 1: /Relay_Control_4/Relay_FeedBack -> /Relay_FeedBack_4
- D1 pad 3: /Voltage_measure_1/VDC_SENSE -> /VDC_1_measure
- D12 pad 1: CAN1_RXD_MCU -> /CAN_RXD_MCU
- D12 pad 2: CAN1_TXD_MCU -> /CAN_TXD_MCU
- D26 pad 3: /Relay_Control_1/Relay_FeedBack -> /Relay_FeedBack_1
- D3 pad 3: Current_SENSE -> /Current_1_measure
- D30 pad 3: /Relay_Control_2/Relay_FeedBack -> /Relay_FeedBack_2
- D34 pad 3: /Relay_Control_3/Relay_FeedBack -> /Relay_FeedBack_3
- D38 pad 3: /Relay_Control_4/Relay_FeedBack -> /Relay_FeedBack_4
- D4 pad 3: Current_SENSE -> /Current_2_measure
- D80 pad 3: /Voltage_measure_3/VDC_SENSE -> /VDC_3_measure
- D9 pad 3: /Voltage_measure_2/VDC_SENSE -> /VDC_2_measure
- H1 pad 1: GND -> GNDD
- H2 pad 1: GND -> GNDD
- J16 pad 1: /Current_measure_1/-15V -> /Current_measure_1/+15V
- J16 pad 2: unconnected-(J16-Pin_2-Pad2) -> /Current_measure_1/-15V
- J16 pad 3: /Current_measure_1/+15V -> /Current_measure_1/M
- J16 pad 4: /Current_measure_1/M -> unconnected-(J16-Pin_4-Pad4)
- J17 pad 1: /Current_measure_2/-15V -> /Current_measure_2/+15V
- J17 pad 2: unconnected-(J17-Pin_2-Pad2) -> /Current_measure_2/-15V
- J17 pad 3: /Current_measure_2/+15V -> /Current_measure_2/M
- J17 pad 4: /Current_measure_2/M -> unconnected-(J17-Pin_4-Pad4)
- L3 pad 1: Net-(C68-Pad1) -> +24V
- R10 pad 2: /Voltage_measure_1/VDC_SENSE -> /VDC_1_measure
- R138 pad 2: /Voltage_measure_3/VDC_SENSE -> /VDC_3_measure
- R18 pad 2: Current_SENSE -> /Current_1_measure
- R45 pad 2: /Voltage_measure_2/VDC_SENSE -> /VDC_2_measure
- R60 pad 1: /Relay_Control_1/Relay_CTRL -> /Relay_Control_1
- R65 pad 1: /Relay_Control_1/Relay_FeedBack -> /Relay_FeedBack_1
- R66 pad 1: /Relay_Control_2/Relay_CTRL -> /Relay_Control_2
- R71 pad 1: /Relay_Control_2/Relay_FeedBack -> /Relay_FeedBack_2
- R72 pad 1: /Relay_Control_3/Relay_CTRL -> /Relay_Control_3
- R77 pad 1: /Relay_Control_3/Relay_FeedBack -> /Relay_FeedBack_3
- R78 pad 1: /Relay_Control_4/Relay_CTRL -> /Relay_Control_4
- R83 pad 1: /Relay_Control_4/Relay_FeedBack -> /Relay_FeedBack_4
- R86 pad 2: Current_SENSE -> /Current_2_measure
- U10 pad 3: /Relay_Control_2/Relay_FeedBack -> /Relay_FeedBack_2
- U12 pad 3: /Relay_Control_3/Relay_FeedBack -> /Relay_FeedBack_3
- U14 pad 3: /Relay_Control_4/Relay_FeedBack -> /Relay_FeedBack_4
- U5 pad 21: /ERROR_LvL1 -> /Current_1_measure
- U5 pad 22: /ERROR_LvL2 -> /Current_2_measure
- U5 pad 23: /ERROR_LvL3 -> unconnected-(U5-PA7-Pad23)
- U5 pad 24: unconnected-(U5-PC4-Pad24) -> /VDC_3_measure
- U5 pad 25: unconnected-(U5-PC5-Pad25) -> /VDC_2_measure
- U5 pad 26: unconnected-(U5-PB0-Pad26) -> /VDC_1_measure
- U5 pad 33: /GPIO1 -> unconnected-(U5-PB12-Pad33)
- U5 pad 34: /GPIO2 -> unconnected-(U5-PB13-Pad34)
- U5 pad 35: /GPIO3 -> unconnected-(U5-PB14-Pad35)
- U5 pad 36: /GPIO4 -> /Relay_FeedBack_4
- U5 pad 37: /GPIO5 -> /Relay_Control_4
- U5 pad 38: /GPIO6 -> /Relay_FeedBack_3
- U5 pad 39: /GPIO7 -> /Relay_Control_3
- U5 pad 40: /GPIO8 -> /Relay_FeedBack_2
- U5 pad 41: unconnected-(U5-PA8-Pad41) -> /Relay_Control_2
- U5 pad 42: /RS_TXD_MCU -> /Relay_FeedBack_1
- U5 pad 43: /RS_RXD_MCU -> /Relay_Control_1
- U5 pad 50: /Solenoid1_MCU -> unconnected-(U5-PA15-Pad50)
- U5 pad 51: /Solenoid2_MCU -> unconnected-(U5-PC10-Pad51)
- U5 pad 52: /Solenoid3_MCU -> unconnected-(U5-PC11-Pad52)
- U5 pad 53: /Solenoid4_MCU -> unconnected-(U5-PC12-Pad53)
- U8 pad 3: /Relay_Control_1/Relay_FeedBack -> /Relay_FeedBack_1
Routing:
- net +5VD: track 0.00 -> 139.8 mm, vias 0 -> 12
- net +5V: track 2.90 -> 133.4 mm, vias 0 -> 22
- net /Relay_Control_1: track 0.00 -> 102.3 mm
- net /Relay_FeedBack_1: track 0.00 -> 92.2 mm
- net GND: track 24.3 -> 106.5 mm, vias 6 -> 80
- net +3.3V: track 22.7 -> 99.8 mm, vias 6 -> 75
- net /VDC_3_measure: track 0.00 -> 73.6 mm
- net /VDC_1_measure: track 0.00 -> 67.5 mm
- net /Relay_Control_2: track 0.00 -> 66.5 mm
- net /VDC_2_measure: track 0.00 -> 65.5 mm
- net /Current_2_measure: track 0.00 -> 60.5 mm, vias 0 -> 1
- net /Relay_FeedBack_2: track 0.00 -> 56.5 mm
- net /Current_1_measure: track 0.00 -> 47.6 mm, vias 0 -> 1
- net /Relay_FeedBack_4: track 0.00 -> 45.1 mm
- net /CAN_RXD_MCU: track 0.00 -> 39.8 mm
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- added copper zone on F.Cu, net +3.3V
- added copper zone on In2.Cu, net +3.3V
- added copper zone on B.Cu, net +5V
- added copper zone on F.Cu, net +5V
- added copper zone on B.Cu, net +5VD
- added copper zone on F.Cu, net +5VD
- added copper zone on B.Cu, net GND
- added copper zone on F.Cu, net GND
- added copper zone on In1.Cu, net GND
- added copper zone on In1.Cu, net GND_CAN
Other:
- outline, holes or cut-outs redrawn
- board text added: "+"
- board text added: "+15V"
- board text added: "-"
- board text added: "-15V"
- board text added: "24V IN"
- board text added: "CAN"
- board text added: "CANH"
- board text added: "CANL"
- board text added: "CGND"
- board text added: "Current Sensors"
- board text added: "HV"
- board text added: "J16"
- board text added: "J17"
- board text added: "J6"
- board text added: "M"
- board text added: "Users LEDs"
- board text added: "VDC+"
- board text added: "VDC-"
- board text added: "X"

Commit message: VER1.0: плата разведена, файлы по плате готовы
Parts:
- added D13: Logo, Logo_My:Logo_Company_1, F.Cu at (374.0, 207.3)
- D10, D6, D81: value TO-3216BC-MYF -> ~
- D12: value TD301MCANFD -> ~
- D16, D7, D83: value S1M -> ~
- Q10, Q9: value BC857 -> ~
- Q7, Q8: value BC847 -> ~
- U10, U11, U12, U13, U14, U7, U8, U9: value PC817 -> ~
- U15: value HT75xx-1-SOT89 -> ~
- U17, U2, U3, U32, U33, U6: value OPA333xxDBV -> ~
- U31, U4: value TLV1117LV33DCYR -> ~
Other:
- board text added: "BAT_VDC"
- board text added: "ECG_VDC"
- board text added: "HV_GND"
- board text added: "INV_VDC"
- board text added: "PDU Control board v1.0"
- board text removed: "VDC+"
- board text removed: "VDC-"
