File: PDU_Container_MCU_PCB.kicad_pcb (KiCad board)
At the start: 4 copper layers, 237.2 x 87.2 mm, 285 parts, among them Y1 16M

Commit message: VER1.0: обновил гербера и BOM
Parts:
- C10, C43, C58: value 0.27u -> 220n
- C23, C25, C48, C52, C54, C62, C64: value 0.1u -> 100n
- R10, R138, R45: value 49.9 -> 120
- R39, R52: value 750 -> 1k
- R57: value 1.1k -> 1k
