File: PDU_Container_MCU_PCB.kicad_sch (KiCad schematic)
At the start: 87 parts, among them U1 TLV431, U15 HT75xx-1-SOT89, U31 TLV1117LV33DCYR, U4 TLV1117LV33DCYR

Commit message: VER1.0: добавил функционалку и расставил все на плате
Parts:
- removed C28, C29, C32, C33, C5: 100n, Capacitor_SMD:C_0805_2012Metric_Pad1.18x1.45mm_HandSolder, symbol Device:C_Small
- removed C31: 4.7u, Capacitor_SMD:C_0805_2012Metric_Pad1.18x1.45mm_HandSolder, symbol Device:C_Small
- removed C50, C51: 2.2u, Capacitor_SMD:C_0805_2012Metric_Pad1.18x1.45mm_HandSolder, symbol Device:C_Small
- removed C6: 1u, Capacitor_SMD:C_0805_2012Metric_Pad1.18x1.45mm_HandSolder, symbol Device:C_Small
- removed D13: (no value), LED_SMD:LED_0805_2012Metric, symbol Device:LED_Small
- removed J2: (no value), Connector_Molex:Molex_Mini-Fit_Jr_5566-04A_2x02_P4.20mm_Vertical, symbol Connector_Generic:Conn_02x02_Odd_Even
- removed R16, R17, R35, R36: 1k, Resistor_SMD:R_0805_2012Metric_Pad1.20x1.40mm_HandSolder, symbol Device:R_Small
- removed TP1, TP2: TestPoint, TestPoint:TestPoint_Loop_D1.80mm_Drill1.0mm_Beaded, symbol Connector:TestPoint
- removed U5: (no value), Package_QFP:LQFP-100_14x14mm_P0.5mm, symbol MCU_ST_STM32F4:STM32F407VETx
- added C13, C15, C65: 100n, Capacitor_SMD:C_0805_2012Metric_Pad1.18x1.45mm_HandSolder, symbol Device:C_Small
- added C21: 2.2u, Capacitor_SMD:C_0805_2012Metric_Pad1.18x1.45mm_HandSolder, symbol Device:C_Small
- added D42: (no value), LED_SMD:LED_0805_2012Metric, symbol Device:LED_Small
- added R11, R14: 10k, Resistor_SMD:R_0805_2012Metric_Pad1.20x1.40mm_HandSolder, symbol Device:R_Small
- added R12, R92: 1k, Resistor_SMD:R_0805_2012Metric_Pad1.20x1.40mm_HandSolder, symbol Device:R_Small
- added R54, R95: 20, Resistor_SMD:R_0805_2012Metric_Pad1.20x1.40mm_HandSolder, symbol Device:R_Small
- added U16: (no value), Package_TO_SOT_SMD:SOT-23-6, symbol Power_Protection:USBLC6-2SC6
- added U5: (no value), Package_QFP:LQFP-64_10x10mm_P0.5mm, symbol MCU_ST_STM32F4:STM32F405RGTx
- C16: value 100n -> 4.7u; Description P/N (none) -> Capacitor SMD 50V
- C17, C18, C26, C3, C30: Description P/N (none) -> Capacitor SMD 50V
- C19: value 100n -> 1u; Description P/N (none) -> Capacitor SMD 50V
- C27: value 100n -> 2.2u; Description P/N (none) -> Capacitor SMD 50V
- C4: value 1u -> 100n; Description P/N (none) -> Capacitor SMD 50V
- D5: Product Name BAS416 -> LBAT54HT1G
- D8: Product Name FYLS-0805UBC -> FYLS-0603UBC
- J1: Function (none) -> SWD; Product Name PLS-4 -> KLS1-207-1-04-S; Purpose SWD -> (none)
- Y1: value (none) -> 16M
Connections:
- net +3.3V: now also C13.1, C15.1, R14.1, U16.5 (VBUS), U5.1 (VBAT), U5.13 (VDDA), U5.19 (VDD), U5.32 (VDD), U5.48 (VDD), U5.64 (VDD); no longer C27.1
- net BOOT0: now also R11.2, U5.60 (BOOT0)
- net GND: now also C13.2, C15.2, C21.2, C65.1, R11.1, R12.2, R92.2, U16.2 (GND), U5.12 (VSSA), U5.18 (VSS), U5.63 (VSS)
- net NRST: now also C65.2, R14.2, U5.7 (NRST)
- net at D8.1 (K): now also R12.1
- net at D8.2 (A): now also U5.3 (PC14)
- net at C30.1, Y1.1: now also U5.6 (PH1)
- net at J1.2 (Pin_2): now also R95.2
- net at J1.3 (Pin_3): now also R54.2
- net at C26.2, Y1.3: now also U5.5 (PH0)
- new net: C27.1, U5.47 (VCAP_2)
- new net: R54.1, U16.4 (I/O2)
- new net: R95.1, U16.6 (I/O1)
- new net: D42.1 (K), R92.1
- new net: D42.2 (A), U5.2 (PC13)
- new net: C21.1, U5.31 (VCAP_1)
- new net CAN_RXD_MCU: U5.44 (PA11)
- new net CAN_TXD_MCU: U5.45 (PA12)
- new net ERROR_LvL1: U5.21 (PA5)
- new net ERROR_LvL2: U5.22 (PA6)
- new net ERROR_LvL3: U5.23 (PA7)
- new net GPIO1: U5.33 (PB12)
- new net GPIO2: U5.34 (PB13)
- new net GPIO3: U5.35 (PB14)
- new net GPIO4: U5.36 (PB15)
- new net GPIO5: U5.37 (PC6)
- new net GPIO6: U5.38 (PC7)
- new net GPIO7: U5.39 (PC8)
- new net GPIO8: U5.40 (PC9)
- new net RS_RXD_MCU: U5.43 (PA10)
- new net RS_TXD_MCU: U5.42 (PA9)
- new net SWCLK: U16.1 (I/O1), U5.49 (PA14)
- new net SWDIO: U16.3 (I/O2), U5.46 (PA13)
- new net Solenoid1_MCU: U5.50 (PA15)
- new net Solenoid2_MCU: U5.51 (PC10)
- new net Solenoid3_MCU: U5.52 (PC11)
- new net Solenoid4_MCU: U5.53 (PC12)
- no-connect marks 58 -> 12
Other:
- sheet Current_measure_1: file Sch/Current_measure.kicad_sch -> Sch\Current_measure.kicad_sch
- sheet Current_measure_2: file Sch/Current_measure.kicad_sch -> Sch\Current_measure.kicad_sch
- sheet Relay_Control_1: file Sch/Power_relay_control.kicad_sch -> Sch\Power_relay_control.kicad_sch
- sheet Relay_Control_2: file Sch/Power_relay_control.kicad_sch -> Sch\Power_relay_control.kicad_sch
- sheet Relay_Control_3: file Sch/Power_relay_control.kicad_sch -> Sch\Power_relay_control.kicad_sch
- sheet Relay_Control_4: file Sch/Power_relay_control.kicad_sch -> Sch\Power_relay_control.kicad_sch
- sheet Voltage_measure_1: file Sch/Voltage_measure.kicad_sch -> Sch\Voltage_measure.kicad_sch
- sheet Voltage_measure_2: file Sch/Voltage_measure.kicad_sch -> Sch\Voltage_measure.kicad_sch
- sheet Voltage_measure_3: file Sch/Voltage_measure.kicad_sch -> Sch\Voltage_measure.kicad_sch
- moved on the sheet: C47, C48, C49, D12, D14, L1, R37, R40

Commit message: VER1.0: оптимизировал схему измерения напряжения
Parts:
- removed R58: 1k, Resistor_SMD:R_0805_2012Metric_Pad1.20x1.40mm_HandSolder, symbol Device:R_Small
- removed U1: TLV431, Package_TO_SOT_SMD:SOT-23, symbol Reference_Voltage:TL431DBZ
- added C5: 100n, Capacitor_SMD:C_0805_2012Metric_Pad1.18x1.45mm_HandSolder, symbol Device:C
- added J35: (no value), Connector_Molex:Molex_Mini-Fit_Jr_5566-04A_2x02_P4.20mm_Vertical, symbol Connector_Generic:Conn_02x02_Odd_Even
- added U17: OPA333xxDBV, Package_TO_SOT_SMD:SOT-23-5, symbol Amplifier_Operational:OPA333xxDBV
- D18: Product Name WRB2403S-3WR2 -> WRB2405S-3WR2
- R23: value 240 -> 23.2k
- R24: value 1k -> 10k
Connections:
- net +1V0: now also U17.1, U17.4 (-); no longer C73.2, R23.2, R24.1
- net +3.3VP: now also R23.1, C5.1, U17.5 (V+)
- net CANH: now also J35.2 (Pin_2)
- net CANL: now also J35.1 (Pin_1)
- net GNDPWR: now also C5.2, U17.2 (V-)
- net GND_CAN: now also J35.3 (Pin_3), J35.4 (Pin_4)
- new net: C73.2, R23.2, R24.1, U17.3 (+)
Other:
- sheet Current_measure_1: file Sch\Current_measure.kicad_sch -> Sch/Current_measure.kicad_sch
- sheet Current_measure_2: file Sch\Current_measure.kicad_sch -> Sch/Current_measure.kicad_sch
- sheet Relay_Control_1: file Sch\Power_relay_control.kicad_sch -> Sch/Power_relay_control.kicad_sch
- sheet Relay_Control_2: file Sch\Power_relay_control.kicad_sch -> Sch/Power_relay_control.kicad_sch
- sheet Relay_Control_3: file Sch\Power_relay_control.kicad_sch -> Sch/Power_relay_control.kicad_sch
- sheet Relay_Control_4: file Sch\Power_relay_control.kicad_sch -> Sch/Power_relay_control.kicad_sch
- sheet Voltage_measure_1: file Sch\Voltage_measure.kicad_sch -> Sch/Voltage_measure.kicad_sch
- sheet Voltage_measure_2: file Sch\Voltage_measure.kicad_sch -> Sch/Voltage_measure.kicad_sch
- sheet Voltage_measure_3: file Sch\Voltage_measure.kicad_sch -> Sch/Voltage_measure.kicad_sch
- note removed: "Разъемы и механические отверстия"
- moved on the sheet: C73, J34, R23, R24

Commit message: VER1.0: плата разведена
Parts:
- removed F2: (no value), Fuse:Fuse_1812_4532Metric, symbol Device:Fuse_Small
Connections:
- net CAN1_RXD_MCU is gone; now on net CAN_RXD_MCU: D12.1 (RXD)
- net CAN1_TXD_MCU is gone; now on net CAN_TXD_MCU: D12.2 (TXD)
- net +24V: now also C68.1, L3.1
- net GND: no longer H1.1, H2.1
- net GNDD: now also H1.1, H2.1
- net VDC_3_measure: now reaches U5.24 (PC4)
- net VDC_2_measure: now reaches U5.25 (PC5)
- net VDC_1_measure: now reaches U5.26 (PB0)
- net Relay_Control_2: now reaches U5.41 (PA8)
- net ERROR_LvL1 renamed Current_1_measure
- net ERROR_LvL2 renamed Current_2_measure
- net ERROR_LvL3: no longer names the net of U5.23 (PA7)
- net GPIO1: no longer names the net of U5.33 (PB12)
- net GPIO2: no longer names the net of U5.34 (PB13)
- net GPIO3: no longer names the net of U5.35 (PB14)
- net GPIO4 renamed Relay_FeedBack_4
- net GPIO5 renamed Relay_Control_4
- net GPIO6 renamed Relay_FeedBack_3
- net GPIO7 renamed Relay_Control_3
- net GPIO8 renamed Relay_FeedBack_2
- net RS_RXD_MCU renamed Relay_Control_1
- net RS_TXD_MCU renamed Relay_FeedBack_1
- net Solenoid1_MCU: no longer names the net of U5.50 (PA15)
- net Solenoid2_MCU: no longer names the net of U5.51 (PC10)
- net Solenoid3_MCU: no longer names the net of U5.52 (PC11)
- net Solenoid4_MCU: no longer names the net of U5.53 (PC12)
Other:
- sheet Current_measure_1 ports: added Current_measure; removed none
- sheet Current_measure_2 ports: added Current_measure; removed none

Commit message: VER1.0: плата разведена, файлы по плате готовы
Parts:
- added D13: Logo, Logo_My:Logo_Company_1, symbol Logo_My:Logo_template
- C34, C35, C36, C37, C38, C39, C44, C47, C48, C49, C5, C71, C72, C73: Description P/N (none) -> Capacitor SMD 50V
- C8: Description P/N (none) -> Polarized capacitor
- D12: value TD301MCANFD -> (none); Product Name (none) -> TD301MCANFD
- D18: Description P/N DC/DC converter -> DC/DC
- J34, J35: Purpose CAN -> (none)
- L1: Description P/N (none) -> Inductor SMD; Product Name (none) -> ACM2520-301-2P-T002
- L2: Description P/N (none) -> Inductor SMD
- R23, R24, R37, R39, R40, R52: Description P/N (none) -> Resistor SMD
- U15: value HT75xx-1-SOT89 -> (none); Description P/N (none) -> Linear regulator
- U17: value OPA333xxDBV -> (none); Description P/N (none) -> Op-Amp; Product Name (none) -> OPA333xxDBV
- U31, U4: value TLV1117LV33DCYR -> (none); Description P/N (none) -> Linear regulator; Product Name (none) -> TLV1117LV33DCYR
Other:
- moved on the sheet: C13, C15, C16, C17, C18, C19, C21, C26, C27, C3, C30, C34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

Commit message: VER1.0: поправил BOM
Parts:
- J6: Product Name DS1073-01-2x2MR3T6 -> DS1073-01-2x2-MVT6
Changed lines of the file:
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@@
 			)
 		)
-		(property "Product Name" "DS1073-01-2x2MR3T6"
+		(property "Product Name" "DS1073-01-2x2-MVT6"
 			(at 44.45 294.64 0)
 			(hide yes)
@@
 			(at 434.34 86.36 0)
 			(hide yes)
+			(show_name no)
+			(do_not_autoplace no)
+			(effects
+				(font
+					(size 1.27 1.27)
+				)
+			)
+		)
+		(property "Function" ""
+			(at 434.34 86.36 0)
+			(hide yes)
