File: PDU_Container_MCU_PCB.kicad_sch (KiCad schematic)
At the start: 83 parts, among them Y1 16M

Commit message: VER1.0: обновил гербера и BOM
Parts:
- C48: value 0.1u -> 100n
- D12: Description P/N (none) -> CAN Transiever
- D42, D8: Product Name FYLS-0603UBC -> FYLS-0805UBC
- R11, R12, R14, R23, R24, R37, R40, R54, R55, R84, R85, R92, R95: Description P/N Resistor SMD -> Resistor SMD 1%
- R39, R52: value 750 -> 1k; Description P/N Resistor SMD -> Resistor SMD 1%
- R57: value 1.1k -> 1k; Description P/N Resistor SMD -> Resistor SMD 1%
- U16: Product Name USBLC6-2P6 -> USBLC6-2SC6
- U17: Product Name OPA333xxDBV -> OPA333
Changed lines of the file:
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@@
 			)
 		)
+		(property "Description P/N" "CAN Transiever"
+			(at 368.3 78.74 0)
+			(hide yes)
+			(show_name no)
+			(do_not_autoplace no)
+			(effects
+				(font
+					(size 1.27 1.27)
+				)
+			)
+		)
 		(pin "6"
 		)
@@
 			)
 		)
-		(property "Product Name" "FYLS-0603UBC"
+		(property "Product Name" "FYLS-0805UBC"
 			(at 97.79 144.78 0)
 			(hide yes)
@@
 			)
 		)
-		(property "Description P/N" "Resistor SMD"
+		(property "Description P/N" "Resistor SMD 1%"
 			(at 88.9 71.12 0)
 			(hide yes)
@@
 			)
 		)
-		(property "Description P/N" "Resistor SMD"
+		(property "Description P/N" "Resistor SMD 1%"
 			(at 110.49 71.12 0)
 			(hide yes)
@@
 			)
 		)
-		(property "Description P/N" "Resistor SMD"
+		(property "Description P/N" "Resistor SMD 1%"
 			(at 388.62 88.9 0)
 			(hide yes)
@@
 			)
 		)
-		(property "Value" "750"
+		(property "Value" "1k"
 			(at 261.62 335.28 0)
 			(show_name no)
@@
 			)
 		)
-		(property "Description P/N" "Resistor SMD"
+		(property "Description P/N" "Resistor SMD 1%"
 			(at 260.35 336.55 0)
 			(hide yes)
@@
 			)
 		)
-		(property "Product Name" "USBLC6-2P6"
+		(property "Product Name" "USBLC6-2SC6"
 			(at 185.42 111.76 0)
 			(hide yes)
@@
 			)
 		)
-		(property "Description P/N" "Resistor SMD"
+		(property "Description P/N" "Resistor SMD 1%"
 			(at 388.62 81.28 0)
 			(hide yes)
@@
 			)
 		)
-		(property "Description P/N" "Resistor SMD"
+		(property "Description P/N" "Resistor SMD 1%"
 			(at 295.91 340.36 0)
 			(hide yes)
@@
 			)
 		)
-		(property "Product Name" "FYLS-0603UBC"
+		(property "Product Name" "FYLS-0805UBC"
 			(at 88.9 144.78 0)
 			(hide yes)
@@
 			)
 		)
-		(property "Description P/N" "Resistor SMD"
+		(property "Description P/N" "Resistor SMD 1%"
 			(at 295.91 327.66 0)
 			(hide yes)
@@
 			)
 		)
-		(property "Description P/N" "Resistor SMD"
+		(property "Description P/N" "Resistor SMD 1%"
 			(at 97.79 149.86 0)
 			(hide yes)
@@
 			)
 		)
-		(property "Description P/N" "Resistor SMD"
+		(property "Description P/N" "Resistor SMD 1%"
 			(at 195.58 109.22 0)
 			(hide yes)
@@
 			)
 		)
-		(property "Description P/N" "Resistor SMD"
+		(property "Description P/N" "Resistor SMD 1%"
 			(at 78.74 289.56 0)
 			(hide yes)
@@
 			)
 		)
-		(property "Product Name" "OPA333xxDBV"
+		(property "Product Name" "OPA333"
 			(at 322.58 334.01 0)
 			(hide yes)
@@
 			)
 		)
-		(property "Description P/N" "Resistor SMD"
+		(property "Description P/N" "Resistor SMD 1%"
 			(at 124.46 297.18 0)
 			(hide yes)
@@
 			)
 		)
-		(property "Description P/N" "Resistor SMD"
+		(property "Description P/N" "Resistor SMD 1%"
 			(at 88.9 149.86 0)
 			(hide yes)
@@
 			)
 		)
-		(property "Value" "750"
+		(property "Value" "1k"
 			(at 278.13 295.91 0)
 			(show_name no)
@@
 			)
 		)
-		(property "Description P/N" "Resistor SMD"
+		(property "Description P/N" "Resistor SMD 1%"
 			(at 276.86 297.18 0)
 			(hide yes)
@@
 			)
 		)
-		(property "Value" "1.1k"
+		(property "Value" "1k"
 			(at 225.425 295.91 0)
 			(show_name no)
@@
 			)
 		)
-		(property "Description P/N" "Resistor SMD"
+		(property "Description P/N" "Resistor SMD 1%"
 			(at 224.155 297.18 0)
 			(hide yes)
@@
 			)
 		)
-		(property "Value" "0.1u"
+		(property "Value" "100n"
 			(at 346.964 95.758 0)
 			(show_name no)
@@
 			)
 		)
-		(property "Description P/N" "Resistor SMD"
+		(property "Description P/N" "Resistor SMD 1%"
 			(at 195.58 111.76 0)
 			(hide yes)
@@
 			)
 		)
-		(property "Description P/N" "Resistor SMD"
+		(property "Description P/N" "Resistor SMD 1%"
 			(at 85.09 298.45 0)
 			(hide yes)
